Commit message: update

File: urdf/cluedo_robot.xacro (robot description, xacro)
@@ -1,6 +1,6 @@
 <?xml version="1.0" ?>
 <robot name="cluedo_robot" xmlns:xacro="https://www.ros.org/wiki/xacro" >
- <xacro:include filename="$(find robot_urdf)/urdf/materials.xacro" />
- <xacro:include filename="$(find robot_urdf)/urdf/cluedo_robot.gazebo" />
+ <xacro:include filename="$(find exprob_ass2)/urdf/materials.xacro" />
+ <xacro:include filename="$(find exprob_ass2)/urdf/cluedo_robot.gazebo" />
  <xacro:macro name="cylinder_inertia" params="mass r l">
     <inertia ixx="${mass*(3*r*r+l*l)/12}" ixy = "0" ixz = "0"
@@ -115,5 +115,5 @@
   <link name="arm_base_link">
   	<inertial>
-  		<mass value="0.1"/>
+  		<mass value="0.5"/>
   		<origin xyz="0 0 0" rpy="0 0 0" />
   		<inertia ixx="0.0000416666667" ixy="0" ixz="0" iyy="0.0000416666667" iyz="0" izz="0.0000416666667"/>
@@ -145,11 +145,11 @@
   	</inertial>
   	<collision>
-  	  <origin xyz="0 0 0" rpy="0 0 0"/>
-      <geometry>
-        <cylinder radius="0.04" length="0.5"/>
-      </geometry>
-  	</collision>
-  	<visual>
-  	  <origin xyz="0 0 0" rpy="0 0 0"/>
+  	  <origin xyz="0 0 0.25" rpy="0 0 0"/>
+      <geometry>
+        <cylinder radius="0.04" length="0.5"/>
+      </geometry>
+  	</collision>
+  	<visual>
+  	  <origin xyz="0 0 0.25" rpy="0 0 0"/>
       <geometry>
         <cylinder radius="0.04" length="0.5"/>
@@ -161,5 +161,5 @@
   	<axis xyz="0 0 1"/>
   	<limit effort="1000.0" lower="-3.14" upper="3.14" velocity="0.2"/>
-  	<origin rpy="0 0 0" xyz="0 0 0.09"/>
+  	<origin rpy="0 0 0" xyz="0 0 0.05"/>
   	<parent link="arm_base_link"/>
   	<child link="arm_link_01"/>
@@ -221,5 +221,5 @@
     <link name="cluedo_link">
   	<inertial>
-  		<mass value="0.025"/>
+  		<mass value="0.01"/>
   		<origin xyz="0 0 0" rpy="0 0 0" />
   		<inertia ixx="0.000010279" ixy="0" ixz="0" iyy="0.000010279" iyz="0" izz="0.000007225"/>
@@ -242,5 +242,5 @@
   	<axis xyz="1 0 0"/>
   	<limit effort="1000.0" lower="-1.8" upper="1.8" velocity="0.5"/>
-  	<origin rpy="0 0 0" xyz="0 0 0.08"/>
+  	<origin rpy="0 0 0" xyz="0 0 0.5"/>
   	<parent link="arm_link_03"/>
   	<child link="cluedo_link"/>

File: urdf/materials.xacro (robot description, xacro)
@@ -1,4 +1,4 @@
 <?xml version="1.0" ?>
-<robot name="m2wr" xmlns:xacro="https://www.ros.org/wiki/xacro" >
+<robot name="cluedo_robot" xmlns:xacro="https://www.ros.org/wiki/xacro" >
   <material name="black">
     <color rgba="0.0 0.0 0.0 1.0"/>

Commit message: update

File: urdf/cluedo_robot.xacro (robot description, xacro)
@@ -140,5 +140,5 @@
   <link name="arm_link_01">
   	<inertial>
-  		<mass value="0.025"/>
+  		<mass value="0.05"/>
   		<origin xyz="0 0 0" rpy="0 0 0" />
   		<inertia ixx="0.000010279" ixy="0" ixz="0" iyy="0.000010279" iyz="0" izz="0.000007225"/>
@@ -167,5 +167,5 @@
     <link name="arm_link_02">
   	<inertial>
-  		<mass value="0.025"/>
+  		<mass value="0.05"/>
   		<origin xyz="0 0 0" rpy="0 0 0" />
   		<inertia ixx="0.000010279" ixy="0" ixz="0" iyy="0.000010279" iyz="0" izz="0.000007225"/>
@@ -194,5 +194,5 @@
       <link name="arm_link_03">
   	<inertial>
-  		<mass value="0.025"/>
+  		<mass value="0.05"/>
   		<origin xyz="0 0 0" rpy="0 0 0" />
   		<inertia ixx="0.000010279" ixy="0" ixz="0" iyy="0.000010279" iyz="0" izz="0.000007225"/>
@@ -221,5 +221,5 @@
     <link name="cluedo_link">
   	<inertial>
-  		<mass value="0.01"/>
+  		<mass value="0.005"/>
   		<origin xyz="0 0 0" rpy="0 0 0" />
   		<inertia ixx="0.000010279" ixy="0" ixz="0" iyy="0.000010279" iyz="0" izz="0.000007225"/>
@@ -248,5 +248,5 @@
 <link name="right_grip_link">
   	<inertial>
-  		<mass value="0.01"/>
+  		<mass value="0.005"/>
   		<origin xyz="0 0 0" rpy="0 0 0" />
   		<inertia ixx="0.000010279" ixy="0" ixz="0" iyy="0.000010279" iyz="0" izz="0.000007225"/>
@@ -275,5 +275,5 @@
   <link name="left_grip_link">
   	<inertial>
-  		<mass value="0.01"/>
+  		<mass value="0.005"/>
   		<origin xyz="0 0 0" rpy="0 0 0" />
   		<inertia ixx="0.000010279" ixy="0" ixz="0" iyy="0.000010279" iyz="0" izz="0.000007225"/>

Commit message: update

File: urdf/cluedo_robot.xacro (robot description, xacro)
@@ -42,5 +42,5 @@
     <pose>0 0 0.1 0 0 0</pose>
     <inertial>
-      <mass value="5"/>
+      <mass value="7"/>
       <origin rpy="0 0 0" xyz="0 0 0.1"/>
       <inertia ixx="0.0395416666667" ixy="0" ixz="0" iyy="0.106208333333" iyz="0" izz="0.106208333333"/>
@@ -140,5 +140,5 @@
   <link name="arm_link_01">
   	<inertial>
-  		<mass value="0.05"/>
+  		<mass value="0.015"/>
   		<origin xyz="0 0 0" rpy="0 0 0" />
   		<inertia ixx="0.000010279" ixy="0" ixz="0" iyy="0.000010279" iyz="0" izz="0.000007225"/>
@@ -167,10 +167,10 @@
     <link name="arm_link_02">
   	<inertial>
-  		<mass value="0.05"/>
-  		<origin xyz="0 0 0" rpy="0 0 0" />
-  		<inertia ixx="0.000010279" ixy="0" ixz="0" iyy="0.000010279" iyz="0" izz="0.000007225"/>
-  	</inertial>
-  	<collision>
-  	  <origin xyz="0 0 0.25" rpy="0 0 0"/>
+  		<mass value="0.015"/>
+  		<origin xyz="0 0 0" rpy="0 0 0" />
+  		<inertia ixx="0.000010279" ixy="0" ixz="0" iyy="0.000010279" iyz="0" izz="0.000007225"/>
+  	</inertial>
+  	<collision>
+  	  <origin xyz="0 0 0.2" rpy="0 0 0"/>
       <geometry>
         <cylinder radius="0.04" length="0.5"/>
@@ -194,10 +194,10 @@
       <link name="arm_link_03">
   	<inertial>
-  		<mass value="0.05"/>
-  		<origin xyz="0 0 0" rpy="0 0 0" />
-  		<inertia ixx="0.000010279" ixy="0" ixz="0" iyy="0.000010279" iyz="0" izz="0.000007225"/>
-  	</inertial>
-  	<collision>
-  	  <origin xyz="0 0 0.25" rpy="0 0 0"/>
+  		<mass value="0.015"/>
+  		<origin xyz="0 0 0" rpy="0 0 0" />
+  		<inertia ixx="0.000010279" ixy="0" ixz="0" iyy="0.000010279" iyz="0" izz="0.000007225"/>
+  	</inertial>
+  	<collision>
+  	  <origin xyz="0 0 0.2" rpy="0 0 0"/>
       <geometry>
         <cylinder radius="0.04" length="0.5"/>
@@ -226,5 +226,5 @@
   	</inertial>
   	<collision>
-  	  <origin xyz="0 0 0.04" rpy="0 0 1.57"/>
+  	  <origin xyz="0 0 0" rpy="0 0 1.57"/>
       <geometry>
         <box size="0.034 0.2 0.08"/>
@@ -248,5 +248,5 @@
 <link name="right_grip_link">
   	<inertial>
-  		<mass value="0.005"/>
+  		<mass value="0.001"/>
   		<origin xyz="0 0 0" rpy="0 0 0" />
   		<inertia ixx="0.000010279" ixy="0" ixz="0" iyy="0.000010279" iyz="0" izz="0.000007225"/>
@@ -275,5 +275,5 @@
   <link name="left_grip_link">
   	<inertial>
-  		<mass value="0.005"/>
+  		<mass value="0.001"/>
   		<origin xyz="0 0 0" rpy="0 0 0" />
   		<inertia ixx="0.000010279" ixy="0" ixz="0" iyy="0.000010279" iyz="0" izz="0.000007225"/>

Commit message: README

File: urdf/cluedo_robot.xacro (robot description, xacro)
@@ -1,6 +1,6 @@
 <?xml version="1.0" ?>
 <robot name="cluedo_robot" xmlns:xacro="https://www.ros.org/wiki/xacro" >
- <xacro:include filename="$(find exprob_ass2)/urdf/materials.xacro" />
- <xacro:include filename="$(find exprob_ass2)/urdf/cluedo_robot.gazebo" />
+ <xacro:include filename="$(find exprob_ass3)/urdf/materials.xacro" />
+ <xacro:include filename="$(find exprob_ass3)/urdf/cluedo_robot.gazebo" />
  <xacro:macro name="cylinder_inertia" params="mass r l">
     <inertia ixx="${mass*(3*r*r+l*l)/12}" ixy = "0" ixz = "0"
@@ -112,4 +112,32 @@
     <child link="laser"/>
   </joint>
+   <link name="camera_link1">
+	    <collision>
+	      <origin xyz="0 0 0.025" rpy="0 0 0"/>
+	      <geometry>
+		<box size="0.05 0.05 0.05"/>
+	      </geometry>
+	    </collision>
+	    <visual>
+	      <origin xyz="0 0 0.025" rpy="0 0 0"/>
+	      <geometry>
+		<box size="0.05 0.05 0.05"/>
+	      </geometry>
+	      <material name="black">
+		<color rgba="1 0 0 1"/>
+	      </material>
+	    </visual>
+	    <inertial>
+	      <mass value="1e-5" />
+	      <origin xyz="0 0 0" rpy="0 0 0"/>
+	      <inertia ixx="1e-6" ixy="0" ixz="0" iyy="1e-6" iyz="0" izz="1e-6" />
+	    </inertial>
+  </link>
+  <joint name="camera_joint1" type="fixed">
+	    <axis xyz="0 1 0" />
+	    <origin xyz="0 0 0.05" rpy="0 0 0"/>
+	    <parent link="laser"/>
+	    <child link="camera_link1"/>
+	 </joint>
 <!--arm definition -->
   <link name="arm_base_link">
@@ -187,5 +215,5 @@
   <joint name="arm_joint_02" type="revolute">
   	<axis xyz="1 0 0"/>
-  	<limit effort="1000.0" lower="-1.8" upper="1.8" velocity="0.2"/>
+  	<limit effort="1000.0" lower="-2.8" upper="2.8" velocity="0.2"/>
   	<origin rpy="0 0 0" xyz="0 0 0.5"/>
   	<parent link="arm_link_01"/>
@@ -214,5 +242,5 @@
   <joint name="arm_joint_03" type="revolute">
   	<axis xyz="1 0 0"/>
-  	<limit effort="1000.0" lower="-1.8" upper="1.8" velocity="0.2"/>
+  	<limit effort="1000.0" lower="-2.8" upper="2.8" velocity="0.2"/>
   	<origin rpy="0 0 0" xyz="0 0 0.5"/>
   	<parent link="arm_link_02"/>
@@ -246,4 +274,32 @@
   	<child link="cluedo_link"/>
   </joint>
+ <link name="camera_link2">
+	    <collision>
+	      <origin xyz="0 0 0.025" rpy="0 0 0"/>
+	      <geometry>
+		<box size="0.05 0.05 0.05"/>
+	      </geometry>
+	    </collision>
+	    <visual>
+	      <origin xyz="0 0 0.025" rpy="0 0 0"/>
+	      <geometry>
+		<box size="0.05 0.05 0.05"/>
+	      </geometry>
+	      <material name="black">
+		<color rgba="1 0 0 1"/>
+	      </material>
+	    </visual>
+	    <inertial>
+	      <mass value="1e-5" />
+	      <origin xyz="0 0 0" rpy="0 0 0"/>
+	      <inertia ixx="1e-6" ixy="0" ixz="0" iyy="1e-6" iyz="0" izz="1e-6" />
+	    </inertial>
+  </link>
+  <joint name="camera_joint2" type="fixed">
+	    <axis xyz="0 1 0" />
+	    <origin xyz="0 0 0.05" rpy="0 0 0"/>
+	    <parent link="cluedo_link"/>
+	    <child link="camera_link2"/>
+	 </joint>
 <link name="right_grip_link">
   	<inertial>

Commit message: final

File: urdf/cluedo_robot.xacro (robot description, xacro)
@@ -1,6 +1,6 @@
 <?xml version="1.0" ?>
 <robot name="cluedo_robot" xmlns:xacro="https://www.ros.org/wiki/xacro" >
- <xacro:include filename="$(find exprob_ass3)/urdf/materials.xacro" />
- <xacro:include filename="$(find exprob_ass3)/urdf/cluedo_robot.gazebo" />
+ <xacro:include filename="$(find exprob_ass2)/urdf/materials.xacro" />
+ <xacro:include filename="$(find exprob_ass2)/urdf/cluedo_robot.gazebo" />
  <xacro:macro name="cylinder_inertia" params="mass r l">
     <inertia ixx="${mass*(3*r*r+l*l)/12}" ixy = "0" ixz = "0"
@@ -112,32 +112,4 @@
     <child link="laser"/>
   </joint>
-   <link name="camera_link1">
-	    <collision>
-	      <origin xyz="0 0 0.025" rpy="0 0 0"/>
-	      <geometry>
-		<box size="0.05 0.05 0.05"/>
-	      </geometry>
-	    </collision>
-	    <visual>
-	      <origin xyz="0 0 0.025" rpy="0 0 0"/>
-	      <geometry>
-		<box size="0.05 0.05 0.05"/>
-	      </geometry>
-	      <material name="black">
-		<color rgba="1 0 0 1"/>
-	      </material>
-	    </visual>
-	    <inertial>
-	      <mass value="1e-5" />
-	      <origin xyz="0 0 0" rpy="0 0 0"/>
-	      <inertia ixx="1e-6" ixy="0" ixz="0" iyy="1e-6" iyz="0" izz="1e-6" />
-	    </inertial>
-  </link>
-  <joint name="camera_joint1" type="fixed">
-	    <axis xyz="0 1 0" />
-	    <origin xyz="0 0 0.05" rpy="0 0 0"/>
-	    <parent link="laser"/>
-	    <child link="camera_link1"/>
-	 </joint>
 <!--arm definition -->
   <link name="arm_base_link">
@@ -215,5 +187,5 @@
   <joint name="arm_joint_02" type="revolute">
   	<axis xyz="1 0 0"/>
-  	<limit effort="1000.0" lower="-2.8" upper="2.8" velocity="0.2"/>
+  	<limit effort="1000.0" lower="-1.8" upper="1.8" velocity="0.2"/>
   	<origin rpy="0 0 0" xyz="0 0 0.5"/>
   	<parent link="arm_link_01"/>
@@ -242,5 +214,5 @@
   <joint name="arm_joint_03" type="revolute">
   	<axis xyz="1 0 0"/>
-  	<limit effort="1000.0" lower="-2.8" upper="2.8" velocity="0.2"/>
+  	<limit effort="1000.0" lower="-1.8" upper="1.8" velocity="0.2"/>
   	<origin rpy="0 0 0" xyz="0 0 0.5"/>
   	<parent link="arm_link_02"/>
@@ -274,32 +246,4 @@
   	<child link="cluedo_link"/>
   </joint>
- <link name="camera_link2">
-	    <collision>
-	      <origin xyz="0 0 0.025" rpy="0 0 0"/>
-	      <geometry>
-		<box size="0.05 0.05 0.05"/>
-	      </geometry>
-	    </collision>
-	    <visual>
-	      <origin xyz="0 0 0.025" rpy="0 0 0"/>
-	      <geometry>
-		<box size="0.05 0.05 0.05"/>
-	      </geometry>
-	      <material name="black">
-		<color rgba="1 0 0 1"/>
-	      </material>
-	    </visual>
-	    <inertial>
-	      <mass value="1e-5" />
-	      <origin xyz="0 0 0" rpy="0 0 0"/>
-	      <inertia ixx="1e-6" ixy="0" ixz="0" iyy="1e-6" iyz="0" izz="1e-6" />
-	    </inertial>
-  </link>
-  <joint name="camera_joint2" type="fixed">
-	    <axis xyz="0 1 0" />
-	    <origin xyz="0 0 0.05" rpy="0 0 0"/>
-	    <parent link="cluedo_link"/>
-	    <child link="camera_link2"/>
-	 </joint>
 <link name="right_grip_link">
   	<inertial>
